Commit message: Working gimbal structure

File: urdf/camera.xacro (robot description, xacro)
@@ -1,12 +1,10 @@
 <?xml version="1.0"?>
-<robot name="camera" xmlns:xacro="http://www.ros.org/wiki/xacro">
- <xacro:property name="pi" value="3.1415926535897931"/>
-    <link name="world"/>
-    <joint name="fix" type="fixed">
-        <parent link="world"/>
-        <child link="camera_link"/>
-        <origin xyz="0 0 0" rpy="0 0 ${pi/2}"/>
-    </joint>
-        <link name="camera_link">
+<robot xmlns:xacro="http://www.ros.org/wiki/xacro">
+    <xacro:property name="pi" value="3.1415926535897931"/>
+    <xacro:macro name="camera_sensor"
+                 params="robot_namespace  camera_suffix parent_link
+                 xyz rpy  horizontal_fov
+                 image_width image_height image_format max_range visualize type mass">
+        <link name="${robot_namespace}/camera_${camera_suffix}_link">
             <collision>
                 <origin xyz="0 0 0" rpy="0 0 0"/>
@@ -22,23 +20,30 @@
             </visual>
             <inertial>
-                <mass value="1"/>
-                <origin xyz="0 0 0" rpy="0 0 0"/>
+                <mass value="${mass}"/>
+                <origin xyz="0 0 0" rpy="0 0 ${pi}"/>
                 <inertia ixx="0.0000001" ixy="0" ixz="0" iyy="0.0000001" iyz="0" izz="0.0000001"/>
             </inertial>
         </link>
-        <gazebo reference="camera_link">
-            <sensor type="camera" name="camera_view">
+        <joint name="${robot_namespace}/gimbal_joint_pitch" type="${type}">
+            <axis xyz="0 1 0"/>
+            <limit effort="10" velocity="1.0" lower="-1.57" upper="1.57"/>
+            <origin xyz="${xyz}" rpy="${rpy}"/>
+            <parent link="${parent_link}"/>
+            <child link="${robot_namespace}/camera_${camera_suffix}_link"/>
+        </joint>
+        <gazebo reference="${robot_namespace}/camera_${camera_suffix}_link">
+            <sensor type="camera" name="${robot_namespace}_camera_${camera_suffix}">
                 <update_rate>30.0</update_rate>
-                <visualize>true</visualize>
-                <camera name="viewer">
-                    <horizontal_fov>${pi/180*18.92}</horizontal_fov>
+                <visualize>${visualize}</visualize>
+                <camera name="${camera_suffix}">
+                    <horizontal_fov>${horizontal_fov}</horizontal_fov>
                     <image>
-                        <width>800</width>
-                        <height>600</height>
-                        <format>R8G8B8</format>
+                        <width>${image_width}</width>
+                        <height>${image_height}</height>
+                        <format>${image_format}</format>
                     </image>
                     <clip>
                         <near>0.02</near>
-                        <far>100</far>
+                        <far>${max_range}</far>
                     </clip>
                     <noise>
@@ -48,10 +53,11 @@
                     </noise>
                 </camera>
-                <plugin name="camera_controller" filename = "libgazebo_ros_camera.so"><!--filename="libgazebo_ros_openni_kinect.so">-->
-                    <robotNamespace>camera</robotNamespace>
+                <plugin name="${robot_namespace}_camera_${camera_suffix}_controller" filename = "libgazebo_ros_camera.so"><!--filename="libgazebo_ros_openni_kinect.so">-->
+                    <robotNamespace>${robot_namespace}</robotNamespace>
                     <alwaysOn>true</alwaysOn>
                     <updateRate>0.0</updateRate>
-                    <cameraName>camera_viewer</cameraName>
-                    <linkName>camera_link</linkName>
+                    <cameraName>camera_${camera_suffix}</cameraName>
+                    <jointName>${robot_namespace}/gimbal_joint_pitch</jointName>
+                    <linkName>${robot_namespace}/camera_link</linkName>
                     <imageTopicName>image_raw</imageTopicName>
                     <cameraInfoTopicName>camera_info</cameraInfoTopicName>
@@ -59,15 +65,32 @@
                     <!--<depthImageCameraInfoTopicName>depth/camera_info</depthImageCameraInfoTopicName>-->
                     <!--<pointCloudTopicName>depth/points</pointCloudTopicName>-->
-                    <frameName>camera_link</frameName>
+                    <frameName>camera_${camera_suffix}_link</frameName>
                     <!--<pointCloudCutoff>0.5</pointCloudCutoff>-->
                     <!--<pointCloudCutoffMax>${max_range}</pointCloudCutoffMax>-->
-                    <hackBaseline>0.07</hackBaseline>
-                    <distortionK1>0.001</distortionK1>
-                    <distortionK2>0.0001</distortionK2>
-                    <distortionK3>0.0</distortionK3>
-                    <distortionT1>0.0002</distortionT1>
-                    <distortionT2>0.0</distortionT2>
+                    <hackBaseline>0.0</hackBaseline>
+                    <distortionK1>0.082318</distortionK1>
+                    <distortionK2>-1.52317</distortionK2>
+                    <distortionK3>16.3747</distortionK3>
+                    <distortionT1>-0.000258164</distortionT1>
+                    <distortionT2>0.00354797</distortionT2>
                 </plugin>
             </sensor>
+            <!--         ros_control plugin -->
+            <plugin name="gazebo_ros_control" filename="libgazebo_ros_control.so">
+                <robotNamespace>/${robot_namespace}</robotNamespace>
+                <robotSimType>gazebo_ros_control/DefaultRobotHWSim</robotSimType>
+                <legacyModeNS>true</legacyModeNS>
+            </plugin>
         </gazebo>
+        <transmission name="tran3">
+            <type>transmission_interface/SimpleTransmission</type>
+            <joint name="${robot_namespace}/gimbal_joint_pitch">
+                <hardwareInterface>hardware_interface/EffortJointInterface</hardwareInterface>
+            </joint>
+            <actuator name="motor3">
+                <hardwareInterface>hardware_interface/EffortJointInterface</hardwareInterface>
+                <mechanicalReduction>1</mechanicalReduction>
+            </actuator>
+        </transmission>
+    </xacro:macro>
 </robot>

File: urdf/generic_gimbal_base.xacro (robot description, xacro)
@@ -2,8 +2,8 @@
 <robot name="generic_gimbal" xmlns:xacro="http://ros.org/wiki/xacro">
     <xacro:property name="PI" value="3.1415926535897931"/>
-    <xacro:property name="parte_1" value="package://gimbal_controller/urdf/meshes/parte_1.dae"/>
-    <xacro:property name="parte_2" value="package://gimbal_controller/urdf/meshes/parte_2.dae"/>
-    <xacro:property name="parte_3" value="package://gimbal_controller/urdf/meshes/parte_3.dae"/>
-    <xacro:include filename="$(find gimbal_controller)/urdf/camera.xacro"/>
+    <xacro:property name="parte_1" value="package://gimbal_controller/urdf/meshes/gimbal_parte_1.dae"/>
+    <xacro:property name="parte_2" value="package://gimbal_controller/urdf/meshes/gimbal_parte_2.dae"/>
+    <xacro:property name="parte_3" value="package://gimbal_controller/urdf/meshes/gimbal_parte_3.dae"/>
+<!--    <xacro:include filename="$(find_gimbal_controller)/urdf/camera.xacro"/>-->
     <xacro:include filename="$(find gimbal_controller)/urdf/component_snippets.xacro"/>
     <xacro:macro name="box_inertia" params="x y z mass">
@@ -18,10 +18,8 @@
                  params="robot_namespace camera_suffix parent_link
                  horizontal_fov image_width image_height image_format
-                 max_range visualize type mass z">
+                 max_range visualize type mass z x">
         <joint name="${robot_namespace}/gimbal_1_joint" type="fixed">
             <axis xyz="1 0 0"/>
-            <!--<limit eff
-            ort="10" velocity="<1.0" lower="-1.57" upper="1.57"/>-->
-            <origin xyz="0 0 ${z}" rpy="0 0 0"/>
+            <origin xyz="${x} 0 ${z}" rpy="0 0 0"/>
             <parent link="${parent_link}"/>
             <child link="${robot_namespace}/gimbal_1_link"/>
@@ -35,5 +33,5 @@
             </collision>
             <visual>
-                <origin xyz="0 0 0" rpy="0 0 {pi/2}"/>
+                <origin xyz="0 0 0" rpy="0 0 ${pi/2}"/>
                 <geometry>
                     <mesh filename="${parte_1}" scale="1 1 1"/>
@@ -41,15 +39,11 @@
             </visual>
             <inertial>
-                <mass value="0.021"/> <!--021-->
+                <mass value="1"/> <!--021-->
                 <origin xyz="0 0 ${z}" rpy="0 0 0"/>
-                <!--                <xacro:box_inertia x="0.1" y="0.1" z="0.1" mass="0.021"/>-->
-<!--                <inertia ixx="34e-7" ixy="0.00" ixz="0.0" iyy="28.7e-6" iyz="0.0" izz="29.6e-6"/>-->
-                <xacro:box_inertia x="0.01" y="0.01" z="0.01" mass="0.02"/>
-            </inertial>
-        </link>
-        <joint name="gimbal_joint_yaw" type="revolute">
+                <xacro:box_inertia x="0.7" y="0.7" z="0.7" mass="0.1"/>
+            </inertial>
+        </link>
+        <joint name="joint_yaw" type="continuous">
             <axis xyz="0 0 1"/>
-            <limit effort="1" velocity="2.0" lower="-2" upper="2"/>
-<!--            <safety_controller k_velocity="10" k_position="15" soft_lower_limit="-2.0" soft_upper_limit="0.5" />-->
             <dynamics damping="0.01" friction="0.0"/>
             <origin xyz="0 0 0" rpy="0 0 0"/>
@@ -71,15 +65,12 @@
             </visual>
             <inertial>
-                <mass value="0.00369"/>
-                <origin xyz="0 0 0" rpy="0 0 0"/>
-                <xacro:box_inertia x="0.01" y="0.01" z="0.01" mass="0.003"/>
-                <!--                <xacro:box_inertia x="0.1" y="0.1" z="0.1" mass="0.00369"/>-->
-<!--                <inertia ixx="13e-7" ixy="0" ixz="0" iyy="19e-7" iyz="0.0" izz="27e-7"/>-->
-            </inertial>
-        </link>
-        <joint name="gimbal_joint_roll" type="continuous">
+                <mass value="1"/>
+                <origin xyz="0 0 0" rpy="0 0 0"/>
+                <xacro:box_inertia x="0.7" y="0.7" z="0.7" mass="0.1"/>
+            </inertial>
+        </link>
+        <joint name="joint_roll" type="continuous">
             <axis xyz="1 0 0"/>
-            <!--            <limit effort="100" velocity="1.0" lower="-1.57" upper="1.57"/>-->
-            <dynamics damping="0.007" friction="0.0"/>
+            <dynamics damping="0.01" friction="0.0"/>
             <origin xyz="-0.048 0 -0.0595" rpy="0 0 0"/>
             <parent link="${robot_namespace}/gimbal_2_link"/>
@@ -100,14 +91,12 @@
             </visual>
             <inertial>
-                <mass value="0.002"/>
-                <origin xyz="0 0 0" rpy="0 0 0"/>
-                <xacro:box_inertia x="0.01" y="0.01" z="0.01" mass="0.002"/>
-<!--                <inertia ixx="14e-7" ixy="0.0" ixz="0.0" iyy="20e-7" iyz="0.0" izz="6e-6"/>-->
-                <!--                <xacro:box_inertia x="0.1" y="0.1" z="0.1" mass="0.002"/>-->
-            </inertial>
-        </link>
-        <joint name="gimbal_joint_pitch" type="continuous">
+                <mass value="0.1"/>
+                <origin xyz="0 0 0" rpy="0 0 0"/>
+                <xacro:box_inertia x="0.7" y="0.7" z="0.7" mass="0.1"/>
+            </inertial>
+        </link>
+        <joint name="joint_pitch" type="continuous">
             <axis xyz="0 1 0"/>
-            <dynamics damping="0.007" friction="0.0"/>
+            <dynamics damping="0.01" friction="0.0"/>
             <origin xyz="0.038 0 0" rpy="0 0 0"/>
             <parent link="${robot_namespace}/gimbal_3_link"/>
@@ -141,22 +130,22 @@
         <link name="camera_link_optical">
         </link>
-<!--         ADIS16448 IMU. -->
-        <xacro:imu_plugin_macro
-                namespace="${robot_namespace}"
-                imu_suffix="camera"
-                parent_link="${robot_namespace}/camera_link"
-                imu_topic="imu1"
-                mass_imu_sensor="0.015"
-                gyroscope_noise_density="0.0003394"
-                gyroscope_random_walk="0.000038785"
-                gyroscope_bias_correlation_time="1000.0"
-                gyroscope_turn_on_bias_sigma="0.0087"
-                accelerometer_noise_density="0.004"
-                accelerometer_random_walk="0.006"
-                accelerometer_bias_correlation_time="300.0"
-                accelerometer_turn_on_bias_sigma="0.1960">
-            <inertia ixx="0.000001" ixy="0.0" ixz="0.0" iyy="0.000001" iyz="0.0" izz="0.000001" />
-            <origin xyz="0 0 0" rpy="0 0 0" />
-        </xacro:imu_plugin_macro>
+<!--&lt;!&ndash;         ADIS16448 IMU. &ndash;&gt;-->
+<!--        <xacro:imu_plugin_macro-->
+<!--                namespace="${robot_namespace}"-->
+<!--                imu_suffix="camera"-->
+<!--                parent_link="${robot_namespace}/camera_link"-->
+<!--                imu_topic="imu1"-->
+<!--                mass_imu_sensor="0.015"-->
+<!--                gyroscope_noise_density="0.0003394"-->
+<!--                gyroscope_random_walk="0.000038785"-->
+<!--                gyroscope_bias_correlation_time="1000.0"-->
+<!--                gyroscope_turn_on_bias_sigma="0.0087"-->
+<!--                accelerometer_noise_density="0.004"-->
+<!--                accelerometer_random_walk="0.006"-->
+<!--                accelerometer_bias_correlation_time="300.0"-->
+<!--                accelerometer_turn_on_bias_sigma="0.1960">-->
+<!--            <inertia ixx="0.000001" ixy="0.0" ixz="0.0" iyy="0.000001" iyz="0.0" izz="0.000001" />-->
+<!--            <origin xyz="0 0 0" rpy="0 0 0" />-->
+<!--        </xacro:imu_plugin_macro>-->
                 <gazebo reference="camera_link_optical">
                     <sensor type="camera" name="camera1">
@@ -184,5 +173,5 @@
                             <alwaysOn>true</alwaysOn>
                             <updateRate>0.0</updateRate>
-                            <cameraName>camera</cameraName>
+                            <cameraName>${robot_namespace}/camera</cameraName>
                             <imageTopicName>image_raw</imageTopicName>
                             <cameraInfoTopicName>camera_info</cameraInfoTopicName>
@@ -206,5 +195,5 @@
         <transmission name="tran1">
             <type>transmission_interface/SimpleTransmission</type>
-            <joint name="gimbal_joint_yaw">
+            <joint name="joint_yaw">
                 <hardwareInterface>hardware_interface/EffortJointInterface</hardwareInterface>
             </joint>
@@ -216,5 +205,5 @@
         <transmission name="tran2">
             <type>transmission_interface/SimpleTransmission</type>
-            <joint name="gimbal_joint_roll">
+            <joint name="joint_roll">
                 <hardwareInterface>hardware_interface/EffortJointInterface</hardwareInterface>
             </joint>
@@ -226,5 +215,5 @@
         <transmission name="tran3">
             <type>transmission_interface/SimpleTransmission</type>
-            <joint name="gimbal_joint_pitch">
+            <joint name="joint_pitch">
                 <hardwareInterface>hardware_interface/EffortJointInterface</hardwareInterface>
             </joint>
