Commit message: Testing robustness

File: urdf/component_snippets.xacro (robot description, xacro)
@@ -9,5 +9,5 @@
       gyroscope_bias_correlation_time gyroscope_turn_on_bias_sigma
       accelerometer_noise_density accelerometer_random_walk
-      accel_bias_correlation_time accelerometer_turn_on_bias_sigma
+      accelerometer_bias_correlation_time accelerometer_turn_on_bias_sigma
       *inertia *origin">
         <!-- IMU link -->
@@ -57,5 +57,5 @@
                     <accelerometerRandomWalk>${accelerometer_random_walk}</accelerometerRandomWalk>
                     <!-- Accelerometer bias correlation time constant [s] -->
-                    <accelerometerBiasCorrelationTime>${accel_bias_correlation_time}</accelerometerBiasCorrelationTime>
+                    <accelerometerBiasCorrelationTime>${accelerometer_bias_correlation_time}</accelerometerBiasCorrelationTime>
                     <!-- Accelerometer turn on bias standard deviation [m/s^2] -->
                     <accelerometerTurnOnBiasSigma>${accelerometer_turn_on_bias_sigma}</accelerometerTurnOnBiasSigma>

File: urdf/generic_gimbal_base.xacro (robot description, xacro)
@@ -18,8 +18,9 @@
                  params="robot_namespace camera_suffix parent_link
                  horizontal_fov image_width image_height image_format
-                 max_range visualize type mass z x">
+                 max_range visualize type mass x y z">
         <joint name="${robot_namespace}/gimbal_1_joint" type="fixed">
             <axis xyz="1 0 0"/>
-            <origin xyz="${x} 0 ${z}" rpy="0 0 0"/>
+            <!--<limit effort="10" velocity="<1.0" lower="-1.57" upper="1.57"/>-->
+            <origin xyz="${x} ${y} ${z}" rpy="0 0 0"/>
             <parent link="${parent_link}"/>
             <child link="${robot_namespace}/gimbal_1_link"/>
@@ -32,19 +33,22 @@
                 </geometry>
             </collision>
-            <visual>
-                <origin xyz="0 0 0" rpy="0 0 ${pi/2}"/>
-                <geometry>
-                    <mesh filename="${parte_1}" scale="1 1 1"/>
-                </geometry>
-            </visual>
-            <inertial>
-                <mass value="1"/> <!--021-->
+            <!--            <visual>-->
+            <!--                <origin xyz="0 0 0" rpy="0 0 ${pi/2}"/>-->
+            <!--                <geometry>-->
+            <!--                    <mesh filename="${parte_1}" scale="1 1 1"/>-->
+            <!--                </geometry>-->
+            <!--            </visual>-->
+            <inertial>
+                <mass value="0.021"/> <!--021-->
                 <origin xyz="0 0 ${z}" rpy="0 0 0"/>
-                <xacro:box_inertia x="0.7" y="0.7" z="0.7" mass="0.1"/>
-            </inertial>
-        </link>
-        <joint name="joint_yaw" type="continuous">
+                <!--                <xacro:box_inertia x="0.1" y="0.1" z="0.1" mass="0.021"/>-->
+                <!--                <inertia ixx="34e-7" ixy="0.00" ixz="0.0" iyy="28.7e-6" iyz="0.0" izz="29.6e-6"/>-->
+                <xacro:box_inertia x="0.01" y="0.01" z="0.01" mass="0.02"/>
+            </inertial>
+        </link>
+        <joint name="gimbal_joint_yaw" type="continuous">
             <axis xyz="0 0 1"/>
-            <dynamics damping="0.01" friction="0.0"/>
+            <!--            <limit effort="100" velocity="1.0" lower="-1.57" upper="1.57"/>-->
+            <dynamics damping="0.007" friction="0.0"/>
             <origin xyz="0 0 0" rpy="0 0 0"/>
             <parent link="${robot_namespace}/gimbal_1_link"/>
@@ -65,12 +69,15 @@
             </visual>
             <inertial>
-                <mass value="1"/>
-                <origin xyz="0 0 0" rpy="0 0 0"/>
-                <xacro:box_inertia x="0.7" y="0.7" z="0.7" mass="0.1"/>
-            </inertial>
-        </link>
-        <joint name="joint_roll" type="continuous">
+                <mass value="0.00369"/>
+                <origin xyz="0 0 0" rpy="0 0 0"/>
+                <xacro:box_inertia x="0.01" y="0.01" z="0.01" mass="0.003"/>
+                <!--                <xacro:box_inertia x="0.1" y="0.1" z="0.1" mass="0.00369"/>-->
+                <!--                <inertia ixx="13e-7" ixy="0" ixz="0" iyy="19e-7" iyz="0.0" izz="27e-7"/>-->
+            </inertial>
+        </link>
+        <joint name="gimbal_joint_roll" type="continuous">
             <axis xyz="1 0 0"/>
-            <dynamics damping="0.01" friction="0.0"/>
+            <!--            <limit effort="100" velocity="1.0" lower="-1.57" upper="1.57"/>-->
+            <dynamics damping="0.007" friction="0.0"/>
             <origin xyz="-0.048 0 -0.0595" rpy="0 0 0"/>
             <parent link="${robot_namespace}/gimbal_2_link"/>
@@ -91,12 +98,14 @@
             </visual>
             <inertial>
-                <mass value="0.1"/>
-                <origin xyz="0 0 0" rpy="0 0 0"/>
-                <xacro:box_inertia x="0.7" y="0.7" z="0.7" mass="0.1"/>
-            </inertial>
-        </link>
-        <joint name="joint_pitch" type="continuous">
+                <mass value="0.002"/>
+                <origin xyz="0 0 0" rpy="0 0 0"/>
+                <xacro:box_inertia x="0.01" y="0.01" z="0.01" mass="0.002"/>
+                <!--                <inertia ixx="14e-7" ixy="0.0" ixz="0.0" iyy="20e-7" iyz="0.0" izz="6e-6"/>-->
+                <!--                <xacro:box_inertia x="0.1" y="0.1" z="0.1" mass="0.002"/>-->
+            </inertial>
+        </link>
+        <joint name="gimbal_joint_pitch" type="continuous">
             <axis xyz="0 1 0"/>
-            <dynamics damping="0.01" friction="0.0"/>
+            <dynamics damping="0.007" friction="0.0"/>
             <origin xyz="0.038 0 0" rpy="0 0 0"/>
             <parent link="${robot_namespace}/gimbal_3_link"/>
@@ -130,70 +139,70 @@
         <link name="camera_link_optical">
         </link>
-<!--&lt;!&ndash;         ADIS16448 IMU. &ndash;&gt;-->
-<!--        <xacro:imu_plugin_macro-->
-<!--                namespace="${robot_namespace}"-->
-<!--                imu_suffix="camera"-->
-<!--                parent_link="${robot_namespace}/camera_link"-->
-<!--                imu_topic="imu1"-->
-<!--                mass_imu_sensor="0.015"-->
-<!--                gyroscope_noise_density="0.0003394"-->
-<!--                gyroscope_random_walk="0.000038785"-->
-<!--                gyroscope_bias_correlation_time="1000.0"-->
-<!--                gyroscope_turn_on_bias_sigma="0.0087"-->
-<!--                accelerometer_noise_density="0.004"-->
-<!--                accelerometer_random_walk="0.006"-->
-<!--                accelerometer_bias_correlation_time="300.0"-->
-<!--                accelerometer_turn_on_bias_sigma="0.1960">-->
-<!--            <inertia ixx="0.000001" ixy="0.0" ixz="0.0" iyy="0.000001" iyz="0.0" izz="0.000001" />-->
-<!--            <origin xyz="0 0 0" rpy="0 0 0" />-->
-<!--        </xacro:imu_plugin_macro>-->
-                <gazebo reference="camera_link_optical">
-                    <sensor type="camera" name="camera1">
-                        <update_rate>30.0</update_rate>
-                        <visualize>${visualize}</visualize>
-                        <camera name="${camera_suffix}">
-                            <horizontal_fov>${horizontal_fov}</horizontal_fov>
-                            <image>
-                                <width>${image_width}</width>
-                                <height>${image_height}</height>
-                                <format>${image_format}</format>
-                            </image>
-                            <clip>
-                                <near>0.02</near>
-                                <far>${max_range}</far>
-                            </clip>
-                            <noise>
-                                <type>gaussian</type>
-                                <mean>0.00</mean>
-                                <stddev>0.007</stddev>
-                            </noise>
-                        </camera>
-                        <plugin name="camera_controller" filename="libgazebo_ros_camera.so"><!--filename="libgazebo_ros_openni_kinect.so">-->
-<!--                            <robotNamespace>${robot_namespace}</robotNamespace>-->
-                            <alwaysOn>true</alwaysOn>
-                            <updateRate>0.0</updateRate>
-                            <cameraName>${robot_namespace}/camera</cameraName>
-                            <imageTopicName>image_raw</imageTopicName>
-                            <cameraInfoTopicName>camera_info</cameraInfoTopicName>
-                            <frameName>camera_link_optical</frameName>
-                            <!-- setting hackBaseline to anything but 0.0 will cause a misalignment
-                     between the gazebo sensor image and the frame it is supposed to
-                     be attached to -->
-                            <hackBaseline>0.0</hackBaseline>
-                            <distortionK1>0.0</distortionK1>
-                            <distortionK2>0.0</distortionK2>
-                            <distortionK3>0.0</distortionK3>
-                            <distortionT1>0.0</distortionT1>
-                            <distortionT2>0.0</distortionT2>
-                            <CxPrime>0</CxPrime>
-                            <Cx>0.0</Cx>
-                            <Cy>0.0</Cy>
-                            <focalLength>0.0</focalLength>
-                        </plugin>
-                    </sensor>
-                </gazebo>
+        <!--         ADIS16448 IMU. -->
+        <xacro:imu_plugin_macro
+                namespace="${robot_namespace}"
+                imu_suffix="camera"
+                parent_link="${robot_namespace}/camera_link"
+                imu_topic="imu1"
+                mass_imu_sensor="0.015"
+                gyroscope_noise_density="0.0003394"
+                gyroscope_random_walk="0.000038785"
+                gyroscope_bias_correlation_time="1000.0"
+                gyroscope_turn_on_bias_sigma="0.0087"
+                accelerometer_noise_density="0.004"
+                accelerometer_random_walk="0.006"
+                accelerometer_bias_correlation_time="300.0"
+                accelerometer_turn_on_bias_sigma="0.1960">
+            <inertia ixx="0.000001" ixy="0.0" ixz="0.0" iyy="0.000001" iyz="0.0" izz="0.000001" />
+            <origin xyz="0 0 0" rpy="0 0 0" />
+        </xacro:imu_plugin_macro>
+        <gazebo reference="camera_link_optical">
+            <sensor type="camera" name="camera1">
+                <update_rate>30.0</update_rate>
+                <visualize>${visualize}</visualize>
+                <camera name="${camera_suffix}">
+                    <horizontal_fov>${horizontal_fov}</horizontal_fov>
+                    <image>
+                        <width>${image_width}</width>
+                        <height>${image_height}</height>
+                        <format>${image_format}</format>
+                    </image>
+                    <clip>
+                        <near>0.02</near>
+                        <far>${max_range}</far>
+                    </clip>
+                    <noise>
+                        <type>gaussian</type>
+                        <mean>0.00</mean>
+                        <stddev>0.007</stddev>
+                    </noise>
+                </camera>
+                <plugin name="camera_controller" filename="libgazebo_ros_camera.so"><!--filename="libgazebo_ros_openni_kinect.so">-->
+                    <!--                            <robotNamespace>${robot_namespace}</robotNamespace>-->
+                    <alwaysOn>true</alwaysOn>
+                    <updateRate>0.0</updateRate>
+                    <cameraName>camera_labmetro</cameraName>
+                    <imageTopicName>image_raw</imageTopicName>
+                    <cameraInfoTopicName>camera_info</cameraInfoTopicName>
+                    <frameName>camera_link_optical</frameName>
+                    <!-- setting hackBaseline to anything but 0.0 will cause a misalignment
+             between the gazebo sensor image and the frame it is supposed to
+             be attached to -->
+                    <hackBaseline>0.0</hackBaseline>
+                    <distortionK1>0.0</distortionK1>
+                    <distortionK2>0.0</distortionK2>
+                    <distortionK3>0.0</distortionK3>
+                    <distortionT1>0.0</distortionT1>
+                    <distortionT2>0.0</distortionT2>
+                    <CxPrime>0</CxPrime>
+                    <Cx>0.0</Cx>
+                    <Cy>0.0</Cy>
+                    <focalLength>0.0</focalLength>
+                </plugin>
+            </sensor>
+        </gazebo>
         <transmission name="tran1">
             <type>transmission_interface/SimpleTransmission</type>
-            <joint name="joint_yaw">
+            <joint name="gimbal_joint_yaw">
                 <hardwareInterface>hardware_interface/EffortJointInterface</hardwareInterface>
             </joint>
@@ -205,5 +214,5 @@
         <transmission name="tran2">
             <type>transmission_interface/SimpleTransmission</type>
-            <joint name="joint_roll">
+            <joint name="gimbal_joint_roll">
                 <hardwareInterface>hardware_interface/EffortJointInterface</hardwareInterface>
             </joint>
@@ -215,5 +224,5 @@
         <transmission name="tran3">
             <type>transmission_interface/SimpleTransmission</type>
-            <joint name="joint_pitch">
+            <joint name="gimbal_joint_pitch">
                 <hardwareInterface>hardware_interface/EffortJointInterface</hardwareInterface>
             </joint>

File: urdf/gimbal_structure.xacro (robot description, xacro)
@@ -2,4 +2,9 @@
 <robot name="gimbal" xmlns:xacro="http://www.ros.org/wiki/xacro">
     <xacro:include filename="$(find gimbal_controller)/urdf/generic_gimbal_base.xacro"/>
+    <xacro:property name="support_height" value="$(arg support_height)"/>
+    <xacro:property name="x_resolution" value="$(arg x_resolution)"/>
+    <xacro:property name="y_resolution" value="$(arg y_resolution)"/>
+    <xacro:property name="h_aov" value="$(arg h_aov)"/>
+    <xacro:property name="visualize" value="$(arg visualize)"/>
     <xacro:property name="pi" value="3.1415926535897931"/>
     <link name="world">
@@ -9,5 +14,5 @@
         <!--<limit eff
         ort="10" velocity="<1.0" lower="-1.57" upper="1.57"/>-->
-        <origin xyz="0 0 0.5" rpy="0 0 0"/>
+        <origin xyz="0 0 ${support_height/2}" rpy="0 0 0"/>
         <parent link="world"/>
         <child link="base_link"/>
@@ -16,15 +21,15 @@
         <colision>
             <geometry>
-                <box size="0.1 0.1 1"/>
+                <box size="0.1 0.1 ${support_height}"/>
             </geometry>
         </colision>
         <visual>
             <geometry>
-                <box size="0.1 0.1 1"/>
+                <box size="0.1 0.1 ${support_height}"/>
             </geometry>
         </visual>
         <inertial>
             <mass value="10"/>
-            <xacro:box_inertia x="0.1" y="0.1" z="1" mass="10"/>
+            <xacro:box_inertia x="0.1" y="0.1" z="${support_height}" mass="10"/>
         </inertial>
     </link>
@@ -33,5 +38,5 @@
         <!--<limit eff
         ort="10" velocity="<1.0" lower="-1.57" upper="1.57"/>-->
-        <origin xyz="0.25 0 0.5" rpy="0 0 0"/>
+        <origin xyz="0.25 0 ${support_height/2}" rpy="0 0 0"/>
         <parent link="base_link"/>
         <child link="base_link_1"/>
@@ -60,16 +65,17 @@
     </gazebo>
     <xacro:generic_gimbal
-            robot_namespace="gimbal"
-            camera_suffix=""
+            robot_namespace="m210"
             parent_link="base_link_1"
-            horizontal_fov="${pi/180*33.31}"
-            image_width="5280"
-            image_height="3956"
+            camera_suffix="labmetro"
+            horizontal_fov="${pi/180*h_aov}"
+            image_width="${x_resolution}"
+            image_height="${y_resolution}"
             image_format="R8G8B8"
             max_range="100"
-            visualize="true"
-            type="fixed"
-            mass="1"
+            visualize="${visualize}"
+            type="continuous"
+            mass="0.036"
             z="-0.05"
+            y="0"
             x="0.25">
     </xacro:generic_gimbal>
